File: kicad/rosalyn-gps/rosalyn-gps.sch (KiCad schematic (older format))
At the start: 8 parts

Commit message: initial schematic done
Parts:
- added C1, C11, C5, C7, C8, C9: 100n, symbol Device:C
- added C10: C, symbol Device:C
- added C12: 220n, symbol Device:C
- added C13: 4,7u, symbol Device:C
- added C14: 10n, symbol Device:C
- added C2: 1u, symbol Device:C
- added C3: 470p, symbol Device:C
- added C4, C6: 10u, symbol Device:C
- added FB1: 200, symbol Device:Ferrite_Bead
- added J1: GpsMag, symbol Connector_Generic:Conn_01x08
- added U1: MIC5219-3.3YM5, Package_TO_SOT_SMD:SOT-23-5, symbol Regulator_Linear:MIC5219-3.3YM5
- added U4: HSCDTD008A, symbol rosalyn-gps:HSCDTD008A
- added U5: HMC5883L, symbol rosalyn-gps:HMC5883L
- L1: renamed from L?; value 22u -> 27n
- R2: renamed from R?; value 22 -> 10
- gave numbers to parts that had none: 6
Connections:
- net +3V3: now also C10.1, C11.1, C4.2, C5.2, C6.1, C7.2, C8.2, C9.2, U1.5 (OUT), U4.2 (AVDD), U4.3 (DVDD), U5.2 (VDD), U5.4 (S1)
- net GND: now also C1.1, C10.2, C11.2, C13.2, C14.1, C2.1, C3.1, C4.1, C5.1, C6.2, C7.1, C8.1, C9.1, J1.1 (Pin_1), U1.2 (GND), U4.1 (VSS), U5.13 (GND), U5.9 (GND)
- net gps_pps: now also J1.7 (Pin_7)
- net gps_rx: now also J1.4 (Pin_4)
- net gps_tx: now also J1.3 (Pin_3)
- net i2c_scl: now also J1.5 (Pin_5), U4.7 (SCL), U5.1 (SCL)
- net i2c_sda: now also J1.6 (Pin_6), U4.8 (SDA), U5.16 (SDA)
- net vbat: now reaches BT1.1 (+), R1.1, U2.22 (V_BCKP)
- net at L1.1, R2.2: now also C14.2
- new net: C1.2, C2.2, FB1.1, U1.1 (IN), U1.3 (EN)
- new net: C3.2, U1.4 (BP)
- new net: C13.1, U5.10 (C1)
- new net: C12.2, U5.12 (SETC)
- new net: C12.1, U5.8 (SETP)
- new net +5V: FB1.2, J1.2 (Pin_2)
- new net mag_drdy: J1.8 (Pin_8), U4.4 (DRDY), U5.15 (DRDY)
- no-connect marks 5 -> 7
Other:
- moved on the sheet: BT1, D1, J2, L1, R1, R2, U2, U3

Commit message: initial pcb layout
Parts:
- BT1: footprint (none) -> rosalyn-gps:MS621FE
- C1, C11, C12, C14, C3, C5, C7, C8, C9: footprint (none) -> Capacitor_SMD:C_0603_1608Metric
- C10: value C -> 100n; footprint (none) -> Capacitor_SMD:C_0603_1608Metric
- C13, C2, C4, C6: footprint (none) -> Capacitor_SMD:C_0805_2012Metric
- D1: footprint (none) -> Diode_SMD:D_SOD-323
- FB1, L1: footprint (none) -> Inductor_SMD:L_0603_1608Metric
- J1: footprint (none) -> Connector_JST:JST_SH_SM08B-SRSS-TB_1x08-1MP_P1.00mm_Horizontal
- J2: footprint (none) -> Connector_Coaxial:SMA_Wurth_60312002114503_Vertical
- R1, R2: footprint (none) -> Resistor_SMD:R_0603_1608Metric
- U3: footprint (none) -> Package_SO:SOIC-8_3.9x4.9mm_P1.27mm
- U4: footprint (none) -> rosalyn-gps:HSCDTD008A
- U5: footprint (none) -> rosalyn-gps:HMC5883L
Connections:
- net i2c_scl: no longer U2.18 (SDA/~SPI_CS), U3.6 (SCL)
- net i2c_sda: no longer U2.19 (SCL/SPI_CLK), U3.5 (SDA)
- removed net mag_drdy: J1.8 (Pin_8), U4.4 (DRDY), U5.15 (DRDY)
- new net gps_scl: U2.18 (SDA/~SPI_CS), U3.6 (SCL)
- new net gps_sda: U2.19 (SCL/SPI_CLK), U3.5 (SDA)
- no-connect marks 7 -> 10
Changed lines of the file:
@@
 Date "2020-12-29"
 Rev "v1.0"
-Comp ""
+Comp "www.2-0.dk"
 Comment1 ""
 Comment2 ""
@@
 F 0 "J2" H 7250 2625 50  0000 L CNN
 F 1 "SMA" H 7250 2534 50  0000 L CNN
-F 2 "" H 7150 2650 50  0001 C CNN
+F 2 "Connector_Coaxial:SMA_Wurth_60312002114503_Vertical" H 7150 2650 50  0001 C CNN
 F 3 " ~" H 7150 2650 50  0001 C CNN
 	1    7150 2650
@@
 F 0 "L1" H 6502 2846 50  0000 L CNN
 F 1 "27n" H 6502 2755 50  0000 L CNN
-F 2 "" H 6450 2800 50  0001 C CNN
+F 2 "Inductor_SMD:L_0603_1608Metric" H 6450 2800 50  0001 C CNN
 F 3 "~" H 6450 2800 50  0001 C CNN
 	1    6450 2800
@@
 F 0 "R2" H 6520 3146 50  0000 L CNN
 F 1 "10" H 6520 3055 50  0000 L CNN
-F 2 "" V 6380 3100 50  0001 C CNN
+F 2 "Resistor_SMD:R_0603_1608Metric" V 6380 3100 50  0001 C CNN
 F 3 "~" H 6450 3100 50  0001 C CNN
 	1    6450 3100
@@
 $EndComp
 Text GLabel 4550 2650 0    50   Output ~ 0
-i2c_scl
+gps_scl
 Text GLabel 4550 2750 0    50   BiDi ~ 0
-i2c_sda
+gps_sda
 NoConn ~ 4550 3150
 NoConn ~ 4550 3350
@@
 F 0 "BT1" H 3518 4596 50  0000 L CNN
 F 1 "MS621FE" H 3518 4505 50  0000 L CNN
-F 2 "" V 3400 4560 50  0001 C CNN
+F 2 "rosalyn-gps:MS621FE" V 3400 4560 50  0001 C CNN
 F 3 "~" V 3400 4560 50  0001 C CNN
 	1    3400 4500
@@
 F 0 "R1" V 2943 4300 50  0000 C CNN
 F 1 "1k" V 3034 4300 50  0000 C CNN
-F 2 "" V 3080 4300 50  0001 C CNN
+F 2 "Resistor_SMD:R_0603_1608Metric" V 3080 4300 50  0001 C CNN
 F 3 "~" H 3150 4300 50  0001 C CNN
 	1    3150 4300
@@
 F 0 "D1" H 2850 4083 50  0000 C CNN
 F 1 "1N5817" H 2850 4174 50  0000 C CNN
-F 2 "" H 2850 4300 50  0001 C CNN
+F 2 "Diode_SMD:D_SOD-323" H 2850 4300 50  0001 C CNN
 F 3 "~" H 2850 4300 50  0001 C CNN
 	1    2850 4300
@@
 F 0 "U3" H 9000 2200 50  0000 C CNN
 F 1 "24LC32" H 9000 2100 50  0000 C CNN
-F 2 "" H 8800 1850 50  0001 C CNN
+F 2 "Package_SO:SOIC-8_3.9x4.9mm_P1.27mm" H 8800 1850 50  0001 C CNN
 F 3 "http://ww1.microchip.com/downloads/en/DeviceDoc/21072G.pdf" H 8800 1850 50  0001 C CNN
 	1    8800 1850
@@
 $EndComp
 Text GLabel 9200 1850 2    50   Input ~ 0
-i2c_scl
+gps_scl
 Text GLabel 9200 1750 2    50   BiDi ~ 0
-i2c_sda
+gps_sda
 Text GLabel 5450 1750 1    50   Output ~ 0
 vcc_rf
@@
 F 0 "FB1" V 2276 5450 50  0000 C CNN
 F 1 "200" V 2367 5450 50  0000 C CNN
-F 2 "" V 2480 5450 50  0001 C CNN
+F 2 "Inductor_SMD:L_0603_1608Metric" V 2480 5450 50  0001 C CNN
 F 3 "~" H 2550 5450 50  0001 C CNN
 	1    2550 5450
@@
 F 0 "C1" H 2785 5554 50  0000 R CNN
 F 1 "100n" H 2785 5645 50  0000 R CNN
-F 2 "" H 2938 5450 50  0001 C CNN
+F 2 "Capacitor_SMD:C_0603_1608Metric" H 2938 5450 50  0001 C CNN
 F 3 "~" H 2900 5600 50  0001 C CNN
 	1    2900 5600
@@
 F 0 "C2" H 3186 5554 50  0000 R CNN
 F 1 "1u" H 3186 5645 50  0000 R CNN
-F 2 "" H 3338 5450 50  0001 C CNN
+F 2 "Capacitor_SMD:C_0805_2012Metric" H 3338 5450 50  0001 C CNN
 F 3 "~" H 3300 5600 50  0001 C CNN
 	1    3300 5600
@@
 F 0 "C3" H 4085 5654 50  0000 R CNN
 F 1 "470p" H 4085 5745 50  0000 R CNN
-F 2 "" H 4238 5550 50  0001 C CNN
+F 2 "Capacitor_SMD:C_0603_1608Metric" H 4238 5550 50  0001 C CNN
 F 3 "~" H 4200 5700 50  0001 C CNN
 	1    4200 5700
@@
 F 0 "C4" H 4535 5554 50  0000 R CNN
 F 1 "10u" H 4535 5645 50  0000 R CNN
-F 2 "" H 4688 5450 50  0001 C CNN
+F 2 "Capacitor_SMD:C_0805_2012Metric" H 4688 5450 50  0001 C CNN
 F 3 "~" H 4650 5600 50  0001 C CNN
 	1    4650 5600
@@
 F 0 "C5" H 4935 5554 50  0000 R CNN
 F 1 "100n" H 4935 5645 50  0000 R CNN
-F 2 "" H 5088 5450 50  0001 C CNN
+F 2 "Capacitor_SMD:C_0603_1608Metric" H 5088 5450 50  0001 C CNN
 F 3 "~" H 5050 5600 50  0001 C CNN
 	1    5050 5600
@@
 F 0 "U4" H 8800 3565 50  0000 C CNN
 F 1 "HSCDTD008A" H 8800 3474 50  0000 C CNN
-F 2 "" H 8750 3100 50  0001 C CNN
+F 2 "rosalyn-gps:HSCDTD008A" H 8750 3100 50  0001 C CNN
 F 3 "https://tech.alpsalpine.com/prod/e/pdf/sensor/geomagnetic/hscd/hscdtd008a_data.pdf" H 8750 3100 50  0001 C CNN
 	1    8800 3100
@@
 F 0 "U5" H 8800 5515 50  0000 C CNN
 F 1 "HMC5883L" H 8800 5424 50  0000 C CNN
-F 2 "" H 8750 5050 50  0001 C CNN
+F 2 "rosalyn-gps:HMC5883L" H 8750 5050 50  0001 C CNN
 F 3 "https://media.digikey.com/pdf/Data%20Sheets/Honeywell%20PDFs/HMC5883L.pdf" H 8750 5050 50  0001 C CNN
 	1    8800 5000
@@
 F 0 "C12" H 9565 5146 50  0000 L CNN
 F 1 "220n" H 9565 5055 50  0000 L CNN
-F 2 "" H 9488 4950 50  0001 C CNN
+F 2 "Capacitor_SMD:C_0603_1608Metric" H 9488 4950 50  0001 C CNN
 F 3 "~" H 9450 5100 50  0001 C CNN
 	1    9450 5100
@@
 F 0 "C13" H 10015 5146 50  0000 L CNN
 F 1 "4,7u" H 10015 5055 50  0000 L CNN
-F 2 "" H 9938 4950 50  0001 C CNN
+F 2 "Capacitor_SMD:C_0805_2012Metric" H 9938 4950 50  0001 C CNN
 F 3 "~" H 9900 5100 50  0001 C CNN
 	1    9900 5100
@@
 P 8900 5600
 F 0 "C10" H 9015 5646 50  0000 L CNN
-F 1 "C" H 9015 5555 50  0000 L CNN
-F 2 "" H 8938 5450 50  0001 C CNN
+F 1 "100n" H 9015 5555 50  0000 L CNN
+F 2 "Capacitor_SMD:C_0603_1608Metric" H 8938 5450 50  0001 C CNN
 F 3 "~" H 8900 5600 50  0001 C CNN
 	1    8900 5600
@@
 F 0 "C8" H 8535 3754 50  0000 R CNN
 F 1 "100n" H 8535 3845 50  0000 R CNN
-F 2 "" H 8688 3650 50  0001 C CNN
+F 2 "Capacitor_SMD:C_0603_1608Metric" H 8688 3650 50  0001 C CNN
 F 3 "~" H 8650 3800 50  0001 C CNN
 	1    8650 3800
@@
 F 0 "C11" H 9065 3846 50  0000 L CNN
 F 1 "100n" H 9065 3755 50  0000 L CNN
-F 2 "" H 8988 3650 50  0001 C CNN
+F 2 "Capacitor_SMD:C_0603_1608Metric" H 8988 3650 50  0001 C CNN
 F 3 "~" H 8950 3800 50  0001 C CNN
 	1    8950 3800
@@
 F 0 "C9" H 8915 1346 50  0000 L CNN
 F 1 "100n" H 8915 1255 50  0000 L CNN
-F 2 "" H 8838 1150 50  0001 C CNN
+F 2 "Capacitor_SMD:C_0603_1608Metric" H 8838 1150 50  0001 C CNN
 F 3 "~" H 8800 1300 50  0001 C CNN
 	1    8800 1300
@@
 F 0 "C7" H 5165 1396 50  0000 L CNN
 F 1 "100n" H 5165 1305 50  0000 L CNN
-F 2 "" H 5088 1200 50  0001 C CNN
+F 2 "Capacitor_SMD:C_0603_1608Metric" H 5088 1200 50  0001 C CNN
 F 3 "~" H 5050 1350 50  0001 C CNN
 	1    5050 1350
@@
 F 0 "C6" H 4735 1304 50  0000 R CNN
 F 1 "10u" H 4735 1395 50  0000 R CNN
-F 2 "" H 4888 1200 50  0001 C CNN
+F 2 "Capacitor_SMD:C_0805_2012Metric" H 4888 1200 50  0001 C CNN
 F 3 "~" H 4850 1350 50  0001 C CNN
 	1    4850 1350
@@
 Text GLabel 2450 2750 2    50   Input ~ 0
 gps_pps
-Text GLabel 2450 2850 2    50   Input ~ 0
-mag_drdy
 $Comp
 L Connector_Generic:Conn_01x08 J1
@@
 F 0 "J1" H 2168 2967 50  0000 C CNN
 F 1 "GpsMag" H 2168 2876 50  0000 C CNN
-F 2 "" H 2250 2450 50  0001 C CNN
+F 2 "Connector_JST:JST_SH_SM08B-SRSS-TB_1x08-1MP_P1.00mm_Horizontal" H 2250 2450 50  0001 C CNN
 F 3 "~" H 2250 2450 50  0001 C CNN
 	1    2250 2450
@@
 	0    1    1    0
 $EndComp
-Text GLabel 8400 3100 0    50   Output ~ 0
-mag_drdy
-Text GLabel 8350 5000 0    50   Output ~ 0
-mag_drdy
 Text GLabel 2700 6350 2    50   Output ~ 0
 vbat
@@
 F 0 "C14" H 6865 3146 50  0000 L CNN
 F 1 "10n" H 6865 3055 50  0000 L CNN
-F 2 "" H 6788 2950 50  0001 C CNN
+F 2 "Capacitor_SMD:C_0603_1608Metric" H 6788 2950 50  0001 C CNN
 F 3 "~" H 6750 3100 50  0001 C CNN
 	1    6750 3100
@@
 	5950 2650 6450 2650
 Connection ~ 6450 2650
+NoConn ~ 2450 2850
+NoConn ~ 8400 3100
+NoConn ~ 8350 5000
 $EndSCHEMATC
